Commit message: hold

File: robot_centric_slam/urdf/hobbit.urdf (robot description, URDF)
Before this commit: robot lio, 10 links, 9 joints
Links:
- removed link camera_link
- removed link camera_optical_link
- removed link imu_link
- removed link os_sensor
- removed link sensor_kit_base_link
- link base_link: mass None -> 20.0; geometry visual mesh filename=../meshes/dae/Cube.004.dae scale=0.66667 0.5 0.5
- link fl_link: geometry collision cylinder length=0.07393 radius=0.13644; visual mesh filename=../meshes/dae/Circle.002.dae scale=0.015 0.015 0.01
- link fr_link: geometry collision cylinder length=0.07393 radius=0.13644; visual mesh filename=../meshes/dae/Circle.001.dae scale=0.015 0.015 0.01
- link rl_link: geometry collision cylinder length=0.07393 radius=0.13644; visual mesh filename=../meshes/dae/Circle.023.dae scale=0.015 0.015 0.01
- link rr_link: geometry collision cylinder length=0.07393 radius=0.13644; visual mesh filename=../meshes/dae/Circle.003.dae scale=0.015 0.015 0.01
Joints:
- removed joint camera_joint
- removed joint camera_optical_joint
- removed joint imu_joint
- removed joint os_joint
- removed joint sensor_kit_base_link_joint
